File: numpad.kicad_pcb (KiCad board)
At the start: 2 copper layers, 76.2 x 95.2 mm, 50 parts, among them J1 HRO-TYPE-C-31-M-12, J3 Conn_01x01_Female, J4 Conn_01x01_Female, J5 Conn_01x01_Female, SW1 SW_Push, SW10 SW_Push, SW11 SW_Push, SW12 SW_Push, SW13 SW_Push, SW14 SW_Push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

Commit message: silkscreen location
Parts:
- renumbered J3 to CLK, J5 to GND, J4 to IO
Changed lines of the file:
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@@
     (tags resistor)
     (attr smd)
-    (fp_text reference R2 (at 0 1.17 90) (layer B.SilkS)
+    (fp_text reference R2 (at -1.29 -1.11 90) (layer B.SilkS)
       (effects (font (size 1 1) (thickness 0.15)) (justify mirror))
     )
@@
     (tags resistor)
     (attr smd)
-    (fp_text reference R1 (at 0 1.17 90) (layer B.SilkS)
+    (fp_text reference R1 (at -1.49 1.3 90) (layer B.SilkS)
       (effects (font (size 1 1) (thickness 0.15)) (justify mirror))
     )
@@
     (tags capacitor)
     (attr smd)
-    (fp_text reference CVR2 (at 0 1.17) (layer B.SilkS)
+    (fp_text reference CVR2 (at -2.885 0.07) (layer B.SilkS)
       (effects (font (size 1 1) (thickness 0.15)) (justify mirror))
     )
@@
     (tags capacitor)
     (attr smd)
-    (fp_text reference C11 (at 0 1.17) (layer B.SilkS)
+    (fp_text reference C11 (at -2.34 0.32) (layer B.SilkS)
       (effects (font (size 1 1) (thickness 0.15)) (justify mirror))
     )
@@
     (tags capacitor)
     (attr smd)
-    (fp_text reference C10 (at 0 1.17) (layer B.SilkS)
+    (fp_text reference C10 (at -2.32 0.14) (layer B.SilkS)
       (effects (font (size 1 1) (thickness 0.15)) (justify mirror))
     )
@@
     (tags capacitor)
     (attr smd)
-    (fp_text reference C9 (at 0 1.17) (layer B.SilkS)
+    (fp_text reference C9 (at 0.345 1.15) (layer B.SilkS)
       (effects (font (size 1 1) (thickness 0.15)) (justify mirror))
     )
@@
     (tags capacitor)
     (attr smd)
-    (fp_text reference C8 (at 0 1.17) (layer B.SilkS)
+    (fp_text reference C8 (at 1.88 0.06) (layer B.SilkS)
       (effects (font (size 1 1) (thickness 0.15)) (justify mirror))
     )
@@
     (tags capacitor)
     (attr smd)
-    (fp_text reference C6 (at 0 1.17 90) (layer B.SilkS)
+    (fp_text reference C6 (at 0.58 1.1 90) (layer B.SilkS)
       (effects (font (size 1 1) (thickness 0.15)) (justify mirror))
     )
@@
     (tags capacitor)
     (attr smd)
-    (fp_text reference C5 (at 0 1.17 90) (layer B.SilkS)
+    (fp_text reference C5 (at 1.91 -0.03 90) (layer B.SilkS)
       (effects (font (size 1 1) (thickness 0.15)) (justify mirror))
     )
@@
     (tags "test point SMD pad")
     (attr virtual)
-    (fp_text reference J5 (at 0 1.648) (layer B.SilkS)
+    (fp_text reference GND (at -0.01375 -1.84625) (layer B.SilkS)
       (effects (font (size 1 1) (thickness 0.15)) (justify mirror))
     )
@@
     (tags "test point SMD pad")
     (attr virtual)
-    (fp_text reference J4 (at 0 1.648) (layer B.SilkS)
+    (fp_text reference IO (at -2.02375 0.13375) (layer B.SilkS)
       (effects (font (size 1 1) (thickness 0.15)) (justify mirror))
     )
@@
     (tags "test point SMD pad")
     (attr virtual)
-    (fp_text reference J3 (at 0 1.648) (layer B.SilkS)
+    (fp_text reference CLK (at 0.01625 2.10375) (layer B.SilkS)
       (effects (font (size 1 1) (thickness 0.15)) (justify mirror))
     )
@@
     (tags "SMD SMT crystal")
     (attr smd)
-    (fp_text reference Y1 (at 0 2.8) (layer B.SilkS)
+    (fp_text reference Y1 (at -1.43 2.71) (layer B.SilkS)
       (effects (font (size 1 1) (thickness 0.15)) (justify mirror))
     )
@@
     (tags SOT-23)
     (attr smd)
-    (fp_text reference U3 (at -2.36365 0.153536) (layer B.SilkS)
+    (fp_text reference U3 (at -0.16 2.74) (layer B.SilkS)
       (effects (font (size 1 1) (thickness 0.15)) (justify mirror))
     )
@@
     (tags "LQFP QFP")
     (attr smd)
-    (fp_text reference U2 (at 0 5.85 90) (layer B.SilkS)
-      (effects (font (size 1 1) (thickness 0.15)) (justify mirror))
-    )
+    (fp_text reference U2 (at 0.866588 5.856179 90) (layer B.SilkS)
+      (effects (font (size 1 1) (thickness 0.15)) (justify mirror))
+    )
